Commit message: added robot w/ ball

File: urdf/turtlebot3_waffle_pi.gazebo.xacro (robot description, xacro)
@@ -2,5 +2,5 @@
 <robot name="turtlebot3_waffle_pi_sim" xmlns:xacro="http://ros.org/wiki/xacro">
   <xacro:arg name="laser_visual"  default="false"/>
-  <xacro:arg name="camera_visual" default="false"/>
+  <xacro:arg name="camera_visual" default="true"/>
   <xacro:arg name="imu_visual"    default="false"/>
   <gazebo reference="base_link">
@@ -167,6 +167,3 @@
     </sensor>
   </gazebo>
-  <gazebo reference="ball_link">
-    <material>Gazebo/FlatBlack</material>
-  </gazebo>
 </robot>

File: urdf/turtlebot3_waffle_pi.urdf.xacro (robot description, xacro)
@@ -30,18 +30,4 @@
                izz="1.4612727e-02" />
     </inertial>
-  </link>
-  <joint name="ball_joint" type="fixed">
-    <parent link="base_link"/>
-    <child link="ball_link"/>
-    <origin xyz="0.0 0.0 0.5" rpy="0 0 0"/>
-  </joint>
-  <link name="ball_link">
-    <collision>
-      <origin xyz="0 0 0" rpy="0 0 0"/>
-      <geometry>
-        <sphere radius="0.2"/>
-      </geometry>
-      <material name="dark"/>
-    </collision>
   </link>
   <joint name="wheel_left_joint" type="continuous">
